Commit message: Set up kinect, write scripted policy without camera, create blob detector

File: src/widowx200_core/widowx200_urdf/wx200.urdf (robot description, URDF)
Before this commit: robot wx200, 13 links, 12 joints
Joints:
- joint wrist_angle: limit lower=-2.1467549799530254 upper=1.7453292519943295 effort=100 velocity=3.141592653589793 -> lower=0.8 upper=1.7453292519943295 effort=100 velocity=3.141592653589793

Commit message: Set up data collection with noise

File: src/widowx200_core/widowx200_urdf/wx200.urdf (robot description, URDF)
Before this commit: robot wx200, 13 links, 12 joints
Joints:
- joint wrist_angle: limit lower=0.8 upper=1.7453292519943295 effort=100 velocity=3.141592653589793 -> lower=-0.20 upper=1.7453292519943295 effort=100 velocity=3.141592653589793
